File: PCBs/kicad/turning-feather/turning-feather.kicad_pcb (KiCad board)
At the start: 2 copper layers, 64.8 x 72.4 mm, 24 parts, among them J1 Out to power switch, J2 Out to RJ45, J3 Buttons/beep, J4 RJ45_Shielded, J5 Spare, U1 TSR 1-2450, U2 MIC4427, U3 MIC4427, U4 ZPT

Commit message: Some cleanup to pcb and schema
Routing:
- net +3V3: track 130.7 -> 126.4 mm
- net Net-(JP1+2-Pad16): track 60.1 -> 63.5 mm
- net Net-(J1-Pad3): track 35.8 -> 38.2 mm
- net Net-(J3-Pad2): track 55.0 -> 56.1 mm
- net +5V: track 92.9 -> 93.9 mm
- net Net-(JP1+2-Pad25): track 41.2 -> 42.2 mm
- net Net-(J2-Pad2): track 118.1 -> 119.0 mm
- net Net-(R4-Pad1): track 56.0 -> 56.7 mm
- net GND: vias 6 -> 7

Commit message: Small cleanups for v0.41
Other:
- board text added: "V0.41"
- board text removed: "V0.40"
Changed lines of the file:
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@@
     (add_net "Net-(D1-Pad2)")
+  )
+  (module turning-feather:ZPT8RD (layer F.Cu)
+    (at 135.128 132.334)
+    (descr ZPT-8RD-2)
+    (tags "Integrated Circuit")
+    (fp_text reference U4 (at 6.5 6.35) (layer F.SilkS)
+      (effects (font (size 1.27 1.27) (thickness 0.254)))
+    )
+    (fp_text value ZPT (at 6.5 4.075) (layer F.SilkS)
+      (effects (font (size 1.27 1.27) (thickness 0.254)))
+    )
+    (fp_line (start -1.75 13.7) (end 14.75 13.7) (layer F.Fab) (width 0.2))
+    (fp_line (start 14.75 13.7) (end 14.75 -5.55) (layer F.Fab) (width 0.2))
+    (fp_line (start 14.75 -5.55) (end -1.75 -5.55) (layer F.Fab) (width 0.2))
+    (fp_line (start -1.75 -5.55) (end -1.75 13.7) (layer F.Fab) (width 0.2))
+    (fp_line (start -2.75 -6.55) (end 15.75 -6.55) (layer F.CrtYd) (width 0.1))
+    (fp_line (start 15.75 -6.55) (end 15.75 14.7) (layer F.CrtYd) (width 0.1))
+    (fp_line (start 15.75 14.7) (end -2.75 14.7) (layer F.CrtYd) (width 0.1))
+    (fp_line (start -2.75 14.7) (end -2.75 -6.55) (layer F.CrtYd) (width 0.1))
+    (fp_line (start -1.75 13.7) (end -1.75 -5.55) (layer F.SilkS) (width 0.1))
+    (fp_line (start -1.75 -5.55) (end 14.75 -5.55) (layer F.SilkS) (width 0.1))
+    (fp_line (start 14.75 -5.55) (end 14.75 13.7) (layer F.SilkS) (width 0.1))
+    (fp_line (start 2 13.7) (end 11 13.7) (layer F.SilkS) (width 0.1))
+    (fp_circle (center 1.143 -3.429) (end 2.413 -4.064) (layer F.SilkS) (width 0.12))
+    (fp_circle (center 1.143 -3.429) (end 1.397 -3.429) (layer F.SilkS) (width 0.12))
+    (pad 1 thru_hole circle (at 0 0) (size 1.8 1.8) (drill 1) (layers *.Cu *.Mask)
+      (net 12 "Net-(U4-Pad1)"))
+    (pad 2 thru_hole circle (at 0 2.54) (size 1.8 1.8) (drill 1) (layers *.Cu *.Mask)
+      (net 2 GND))
+    (pad 3 thru_hole circle (at 0 5.08) (size 1.8 1.8) (drill 1) (layers *.Cu *.Mask)
+      (net 2 GND))
+    (pad 4 thru_hole circle (at 0 7.62) (size 1.8 1.8) (drill 1) (layers *.Cu *.Mask)
+      (net 5 +3V3))
+    (pad 5 thru_hole circle (at 0 10.16) (size 1.8 1.8) (drill 1) (layers *.Cu *.Mask)
+      (net 14 "Net-(R4-Pad1)"))
+    (pad 6 thru_hole circle (at 0 12.7) (size 1.8 1.8) (drill 1) (layers *.Cu *.Mask)
+      (net 29 "Net-(JP1+2-Pad14)"))
+    (pad 7 thru_hole circle (at 13 12.7) (size 1.8 1.8) (drill 1) (layers *.Cu *.Mask)
+      (net 13 "Net-(U4-Pad7)"))
+    (pad 8 thru_hole circle (at 13 10.16) (size 1.8 1.8) (drill 1) (layers *.Cu *.Mask)
+      (net 2 GND))
+    (pad 9 thru_hole circle (at 13 7.62) (size 1.8 1.8) (drill 1) (layers *.Cu *.Mask)
+      (net 23 "Net-(JP1+2-Pad7)"))
+    (pad 10 thru_hole circle (at 13 5.08) (size 1.8 1.8) (drill 1) (layers *.Cu *.Mask)
+      (net 35 "Net-(JP1+2-Pad23)"))
+    (pad 11 thru_hole circle (at 13 2.54) (size 1.8 1.8) (drill 1) (layers *.Cu *.Mask)
+      (net 31 "Net-(JP1+2-Pad16)"))
+    (pad 12 thru_hole circle (at 13 0) (size 1.8 1.8) (drill 1) (layers *.Cu *.Mask)
+      (net 25 "Net-(JP1+2-Pad10)"))
+    (model ZPT-8RD.stp
+      (at (xyz 0 0 0))
+      (scale (xyz 1 1 1))
+      (rotate (xyz 0 0 0))
+    )
   )
   (module turning-feather:RJ45_Horizontal_Shielded (layer B.Cu)
@@
       (net 14 "Net-(R4-Pad1)"))
     (model ${KISYS3DMOD}/Button_Switch_THT.3dshapes/SW_PUSH_6mm_H5mm.wrl
-      (at (xyz 0 0 0))
-      (scale (xyz 1 1 1))
-      (rotate (xyz 0 0 0))
-    )
-  )
-  (module turning-feather:ZPT8RD (layer F.Cu)
-    (at 135.128 132.334)
-    (descr ZPT-8RD-2)
-    (tags "Integrated Circuit")
-    (fp_text reference U4 (at 6.5 6.35) (layer F.SilkS)
-      (effects (font (size 1.27 1.27) (thickness 0.254)))
-    )
-    (fp_text value ZPT (at 6.5 4.075) (layer F.SilkS)
-      (effects (font (size 1.27 1.27) (thickness 0.254)))
-    )
-    (fp_line (start -1.75 13.7) (end 14.75 13.7) (layer F.Fab) (width 0.2))
-    (fp_line (start 14.75 13.7) (end 14.75 -5.55) (layer F.Fab) (width 0.2))
-    (fp_line (start 14.75 -5.55) (end -1.75 -5.55) (layer F.Fab) (width 0.2))
-    (fp_line (start -1.75 -5.55) (end -1.75 13.7) (layer F.Fab) (width 0.2))
-    (fp_line (start -2.75 -6.55) (end 15.75 -6.55) (layer F.CrtYd) (width 0.1))
-    (fp_line (start 15.75 -6.55) (end 15.75 14.7) (layer F.CrtYd) (width 0.1))
-    (fp_line (start 15.75 14.7) (end -2.75 14.7) (layer F.CrtYd) (width 0.1))
-    (fp_line (start -2.75 14.7) (end -2.75 -6.55) (layer F.CrtYd) (width 0.1))
-    (fp_line (start -1.75 13.7) (end -1.75 -5.55) (layer F.SilkS) (width 0.1))
-    (fp_line (start -1.75 -5.55) (end 14.75 -5.55) (layer F.SilkS) (width 0.1))
-    (fp_line (start 14.75 -5.55) (end 14.75 13.7) (layer F.SilkS) (width 0.1))
-    (fp_line (start 2 13.7) (end 11 13.7) (layer F.SilkS) (width 0.1))
-    (fp_circle (center 1.143 -3.429) (end 2.413 -4.064) (layer F.SilkS) (width 0.12))
-    (fp_circle (center 1.143 -3.429) (end 1.397 -3.429) (layer F.SilkS) (width 0.12))
-    (pad 1 thru_hole circle (at 0 0) (size 1.8 1.8) (drill 1.2) (layers *.Cu *.Mask)
-      (net 12 "Net-(U4-Pad1)"))
-    (pad 2 thru_hole circle (at 0 2.54) (size 1.8 1.8) (drill 1.2) (layers *.Cu *.Mask)
-      (net 2 GND))
-    (pad 3 thru_hole circle (at 0 5.08) (size 1.8 1.8) (drill 1.2) (layers *.Cu *.Mask)
-      (net 2 GND))
-    (pad 4 thru_hole circle (at 0 7.62) (size 1.8 1.8) (drill 1.2) (layers *.Cu *.Mask)
-      (net 5 +3V3))
-    (pad 5 thru_hole circle (at 0 10.16) (size 1.8 1.8) (drill 1.2) (layers *.Cu *.Mask)
-      (net 14 "Net-(R4-Pad1)"))
-    (pad 6 thru_hole circle (at 0 12.7) (size 1.8 1.8) (drill 1.2) (layers *.Cu *.Mask)
-      (net 29 "Net-(JP1+2-Pad14)"))
-    (pad 7 thru_hole circle (at 13 12.7) (size 1.8 1.8) (drill 1.2) (layers *.Cu *.Mask)
-      (net 13 "Net-(U4-Pad7)"))
-    (pad 8 thru_hole circle (at 13 10.16) (size 1.8 1.8) (drill 1.2) (layers *.Cu *.Mask)
-      (net 2 GND))
-    (pad 9 thru_hole circle (at 13 7.62) (size 1.8 1.8) (drill 1.2) (layers *.Cu *.Mask)
-      (net 23 "Net-(JP1+2-Pad7)"))
-    (pad 10 thru_hole circle (at 13 5.08) (size 1.8 1.8) (drill 1.2) (layers *.Cu *.Mask)
-      (net 35 "Net-(JP1+2-Pad23)"))
-    (pad 11 thru_hole circle (at 13 2.54) (size 1.8 1.8) (drill 1.2) (layers *.Cu *.Mask)
-      (net 31 "Net-(JP1+2-Pad16)"))
-    (pad 12 thru_hole circle (at 13 0) (size 1.8 1.8) (drill 1.2) (layers *.Cu *.Mask)
-      (net 25 "Net-(JP1+2-Pad10)"))
-    (model ZPT-8RD.stp
       (at (xyz 0 0 0))
       (scale (xyz 1 1 1))
@@
     (arrow2b (pts (xy 104.648 78.74) (xy 105.774504 78.153579)))
   )
-  (gr_text V0.40 (at 106.68 120.142 90) (layer F.SilkS)
+  (gr_text V0.41 (at 106.68 120.142 90) (layer F.SilkS)
     (effects (font (size 1 1) (thickness 0.15)))
   )
